File: pcb_design/pcb_design.kicad_pcb (KiCad board)
At the start: 2 copper layers, 360 x 125 mm, 211 parts, among them U1 AVR_CNANO

Commit message: added pictures, gitignore, readme ish done
Parts:
- moved MX3 0.08 mm to (113.9, 70.0)
Connections:
- LED1 pad 3: LED_pin -> VSS
- LED1 pad 4: VSS -> LED_pin
- LED10 pad 3: Net-(LED10-DIN) -> VSS
- LED10 pad 4: VSS -> Net-(LED10-VSS)
- LED11 pad 3: Net-(LED10-DOUT) -> VSS
- LED11 pad 4: VSS -> Net-(LED10-DOUT)
- LED12 pad 3: Net-(LED11-DOUT) -> VSS
- LED12 pad 4: VSS -> Net-(LED11-DOUT)
- LED13 pad 3: Net-(LED12-DOUT) -> VSS
- LED13 pad 4: VSS -> Net-(LED12-DOUT)
- LED14 pad 3: Net-(LED13-DOUT) -> VSS
- LED14 pad 4: VSS -> Net-(LED13-DOUT)
- LED15 pad 3: Net-(LED14-DOUT) -> VSS
- LED15 pad 4: VSS -> Net-(LED14-DOUT)
- LED16 pad 3: Net-(LED15-DOUT) -> VSS
- LED16 pad 4: VSS -> Net-(LED15-DOUT)
- LED17 pad 3: Net-(LED16-DOUT) -> VSS
- LED17 pad 4: VSS -> Net-(LED16-DOUT)
- LED18 pad 3: Net-(LED17-DOUT) -> VSS
- LED18 pad 4: VSS -> Net-(LED17-DOUT)
- LED19 pad 3: Net-(LED18-DOUT) -> VSS
- LED19 pad 4: VSS -> Net-(LED18-DOUT)
- LED2 pad 3: Net-(LED1-DOUT) -> VSS
- LED2 pad 4: VSS -> Net-(LED1-DOUT)
- LED20 pad 3: Net-(LED19-DOUT) -> VSS
- LED20 pad 4: VSS -> Net-(LED19-DOUT)
- LED21 pad 3: Net-(LED20-DOUT) -> VSS
- LED21 pad 4: VSS -> Net-(LED20-DOUT)
- LED22 pad 3: Net-(LED21-DOUT) -> VSS
- LED22 pad 4: VSS -> Net-(LED21-DOUT)
- LED23 pad 3: Net-(LED22-DOUT) -> VSS
- LED23 pad 4: VSS -> Net-(LED22-DOUT)
- LED24 pad 3: Net-(LED23-DOUT) -> VSS
- LED24 pad 4: VSS -> Net-(LED23-DOUT)
- LED25 pad 3: Net-(LED24-DOUT) -> VSS
- LED25 pad 4: VSS -> Net-(LED24-DOUT)
- LED26 pad 3: Net-(LED25-DOUT) -> VSS
- LED26 pad 4: VSS -> Net-(LED25-DOUT)
- LED27 pad 3: Net-(LED26-DOUT) -> VSS
- LED27 pad 4: VSS -> Net-(LED26-DOUT)
- LED28 pad 3: Net-(LED27-DOUT) -> VSS
- LED28 pad 4: VSS -> Net-(LED27-DOUT)
- LED29 pad 3: Net-(LED28-DOUT) -> VSS
- LED29 pad 4: VSS -> Net-(LED28-DOUT)
- LED3 pad 3: Net-(LED2-DOUT) -> VSS
- LED3 pad 4: VSS -> Net-(LED2-DOUT)
- LED30 pad 3: Net-(LED29-DOUT) -> VSS
- LED30 pad 4: VSS -> Net-(LED29-DOUT)
- LED31 pad 3: Net-(LED30-DOUT) -> VSS
- LED31 pad 4: VSS -> Net-(LED30-DOUT)
- LED32 pad 3: Net-(LED31-DOUT) -> VSS
- LED32 pad 4: VSS -> Net-(LED31-DOUT)
- LED33 pad 3: Net-(LED32-DOUT) -> VSS
- LED33 pad 4: VSS -> Net-(LED32-DOUT)
- LED34 pad 3: Net-(LED33-DOUT) -> VSS
- LED34 pad 4: VSS -> Net-(LED33-DOUT)
- LED35 pad 3: Net-(LED34-DOUT) -> VSS
- LED35 pad 4: VSS -> Net-(LED34-DOUT)
- LED36 pad 3: Net-(LED35-DOUT) -> VSS
- LED36 pad 4: VSS -> Net-(LED35-DOUT)
- LED37 pad 3: Net-(LED36-DOUT) -> VSS
- LED37 pad 4: VSS -> Net-(LED36-DOUT)
- LED38 pad 3: Net-(LED37-DOUT) -> VSS
- LED38 pad 4: VSS -> Net-(LED37-DOUT)
- LED39 pad 3: Net-(LED38-DOUT) -> VSS
- LED39 pad 4: VSS -> Net-(LED38-DOUT)
- LED4 pad 3: Net-(LED3-DOUT) -> VSS
- LED4 pad 4: VSS -> Net-(LED3-DOUT)
- LED40 pad 3: Net-(LED39-DOUT) -> VSS
- LED40 pad 4: VSS -> Net-(LED39-DOUT)
- LED41 pad 3: Net-(LED40-DOUT) -> VSS
- LED41 pad 4: VSS -> Net-(LED40-DOUT)
- LED42 pad 3: Net-(LED41-DOUT) -> VSS
- LED42 pad 4: VSS -> Net-(LED41-DOUT)
- LED43 pad 3: Net-(LED42-DOUT) -> VSS
- LED43 pad 4: VSS -> Net-(LED42-DOUT)
- LED44 pad 3: Net-(LED43-DOUT) -> VSS
- LED44 pad 4: VSS -> Net-(LED43-DOUT)
- LED45 pad 3: Net-(LED44-DOUT) -> VSS
- LED45 pad 4: VSS -> Net-(LED44-DOUT)
- LED46 pad 3: Net-(LED45-DOUT) -> VSS
- LED46 pad 4: VSS -> Net-(LED45-DOUT)
- LED47 pad 3: Net-(LED46-DOUT) -> VSS
- LED47 pad 4: VSS -> Net-(LED46-DOUT)
- LED48 pad 3: Net-(LED47-DOUT) -> VSS
- LED48 pad 4: VSS -> Net-(LED47-DOUT)
- LED49 pad 3: Net-(LED48-DOUT) -> VSS
- LED49 pad 4: VSS -> Net-(LED48-DOUT)
- LED5 pad 3: Net-(LED4-DOUT) -> VSS
- LED5 pad 4: VSS -> Net-(LED4-DOUT)
- LED50 pad 3: Net-(LED49-DOUT) -> VSS
- LED50 pad 4: VSS -> Net-(LED49-DOUT)
- LED51 pad 3: Net-(LED50-DOUT) -> VSS
- LED51 pad 4: VSS -> Net-(LED50-DOUT)
- LED52 pad 3: Net-(LED51-DOUT) -> VSS
- LED52 pad 4: VSS -> Net-(LED51-DOUT)
- LED53 pad 3: Net-(LED52-DOUT) -> VSS
- LED53 pad 4: VSS -> Net-(LED52-DOUT)
- LED54 pad 3: Net-(LED53-DOUT) -> VSS
- LED54 pad 4: VSS -> Net-(LED53-DOUT)
- LED55 pad 3: Net-(LED54-DOUT) -> VSS
- LED55 pad 4: VSS -> Net-(LED54-DOUT)
- LED56 pad 3: Net-(LED55-DOUT) -> VSS
- LED56 pad 4: VSS -> Net-(LED55-DOUT)
- LED57 pad 3: Net-(LED56-DOUT) -> VSS
- LED57 pad 4: VSS -> Net-(LED56-DOUT)
- LED58 pad 3: Net-(LED57-DOUT) -> VSS
- LED58 pad 4: VSS -> Net-(LED57-DOUT)
- LED59 pad 3: Net-(LED58-DOUT) -> VSS
- LED59 pad 4: VSS -> Net-(LED58-DOUT)
- LED6 pad 3: Net-(LED5-DOUT) -> VSS
- LED6 pad 4: VSS -> Net-(LED5-DOUT)
- LED60 pad 3: Net-(LED59-DOUT) -> VSS
- LED60 pad 4: VSS -> Net-(LED59-DOUT)
- LED61 pad 3: Net-(LED60-DOUT) -> VSS
- LED61 pad 4: VSS -> Net-(LED60-DOUT)
- LED62 pad 3: Net-(LED61-DOUT) -> VSS
- LED62 pad 4: VSS -> Net-(LED61-DOUT)
- LED63 pad 3: Net-(LED62-DOUT) -> VSS
- LED63 pad 4: VSS -> Net-(LED62-DOUT)
- LED64 pad 3: Net-(LED63-DOUT) -> VSS
- LED64 pad 4: VSS -> Net-(LED63-DOUT)
- LED65 pad 3: Net-(LED64-DOUT) -> VSS
- LED65 pad 4: VSS -> Net-(LED64-DOUT)
- LED66 pad 3: Net-(LED65-DOUT) -> VSS
- LED66 pad 4: VSS -> Net-(LED65-DOUT)
- LED67 pad 3: Net-(LED66-DOUT) -> VSS
- LED67 pad 4: VSS -> Net-(LED66-DOUT)
- LED68 pad 3: Net-(LED67-DOUT) -> VSS
- LED68 pad 4: VSS -> Net-(LED67-DOUT)
- LED69 pad 3: Net-(LED68-DOUT) -> VSS
- LED69 pad 4: VSS -> Net-(LED68-DOUT)
- LED7 pad 3: Net-(LED6-DOUT) -> VSS
- LED7 pad 4: VSS -> Net-(LED6-DOUT)
- LED8 pad 3: Net-(LED7-DOUT) -> VSS
- LED8 pad 4: VSS -> Net-(LED7-DOUT)
- LED9 pad 2: Net-(LED10-DIN) -> Net-(LED10-VSS)
- LED9 pad 3: Net-(LED8-DOUT) -> VSS
- LED9 pad 4: VSS -> Net-(LED8-DOUT)
Routing:
- net VSS: track 1664.2 -> 1515.9 mm, vias 76 -> 77
- net Net-(LED44-DOUT): track 312.8 -> 338.9 mm
- net Net-(LED59-DOUT): track 298.7 -> 318.3 mm
- net Net-(LED30-DOUT): track 318.1 -> 337.0 mm
- net Net-(LED10-VSS): track 0.00 -> 14.7 mm, vias 0 -> 2
- net Net-(LED10-DIN): track 13.6 -> 0.00 mm, vias 2 -> 0
- net Net-(LED15-DOUT): track 302.8 -> 311.8 mm
- net Net-(LED18-DOUT): track 13.9 -> 16.1 mm
- net Net-(LED49-DOUT): track 14.1 -> 15.7 mm
- net Net-(LED45-DOUT): track 16.7 -> 18.3 mm
- net LED_pin: track 58.3 -> 59.9 mm, vias 2 -> 4
- net Net-(LED40-DOUT): track 14.6 -> 16.0 mm
- net Net-(LED2-DOUT): track 14.1 -> 15.4 mm
- net Net-(LED56-DOUT): track 21.5 -> 22.8 mm
- net Net-(LED22-DOUT): track 14.7 -> 16.0 mm
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