File: pcb_design/pcb_design.kicad_sch (KiCad schematic)
At the start: 211 parts, among them U1 AVR_CNANO

Commit message: added pictures, gitignore, readme ish done
Connections:
- net LED_pin: now also LED1.4 (DIN); no longer LED1.3 (DIN)
- net VSS: now also LED1.3 (VSS), LED10.3 (VSS), LED11.3 (VSS), LED12.3 (VSS), LED13.3 (VSS), LED14.3 (VSS), LED15.3 (VSS), LED16.3 (VSS), LED17.3 (VSS), LED18.3 (VSS), LED19.3 (VSS), LED2.3 (VSS), LED20.3 (VSS), LED21.3 (VSS), LED22.3 (VSS), LED23.3 (VSS), LED24.3 (VSS), LED25.3 (VSS), LED26.3 (VSS), LED27.3 (VSS), LED28.3 (VSS), LED29.3 (VSS), LED3.3 (VSS), LED30.3 (VSS), LED31.3 (VSS), LED32.3 (VSS), LED33.3 (VSS), LED34.3 (VSS), LED35.3 (VSS), LED36.3 (VSS), LED37.3 (VSS), LED38.3 (VSS), LED39.3 (VSS), LED4.3 (VSS), LED40.3 (VSS), LED41.3 (VSS), LED42.3 (VSS), LED43.3 (VSS), LED44.3 (VSS), LED45.3 (VSS), LED46.3 (VSS), LED47.3 (VSS), LED48.3 (VSS), LED49.3 (VSS), LED5.3 (VSS), LED50.3 (VSS), LED51.3 (VSS), LED52.3 (VSS), LED53.3 (VSS), LED54.3 (VSS), LED55.3 (VSS), LED56.3 (VSS), LED57.3 (VSS), LED58.3 (VSS), LED59.3 (VSS), LED6.3 (VSS), LED60.3 (VSS), LED61.3 (VSS), LED62.3 (VSS), LED63.3 (VSS), LED64.3 (VSS), LED65.3 (VSS), LED66.3 (VSS), LED67.3 (VSS), LED68.3 (VSS), LED69.3 (VSS), LED7.3 (VSS), LED8.3 (VSS), LED9.3 (VSS); no longer LED1.4 (VSS), LED10.4 (VSS), LED11.4 (VSS), LED12.4 (VSS), LED13.4 (VSS), LED14.4 (VSS), LED15.4 (VSS), LED16.4 (VSS), LED17.4 (VSS), LED18.4 (VSS), LED19.4 (VSS), LED2.4 (VSS), LED20.4 (VSS), LED21.4 (VSS), LED22.4 (VSS), LED23.4 (VSS), LED24.4 (VSS), LED25.4 (VSS), LED26.4 (VSS), LED27.4 (VSS), LED28.4 (VSS), LED29.4 (VSS), LED3.4 (VSS), LED30.4 (VSS), LED31.4 (VSS), LED32.4 (VSS), LED33.4 (VSS), LED34.4 (VSS), LED35.4 (VSS), LED36.4 (VSS), LED37.4 (VSS), LED38.4 (VSS), LED39.4 (VSS), LED4.4 (VSS), LED40.4 (VSS), LED41.4 (VSS), LED42.4 (VSS), LED43.4 (VSS), LED44.4 (VSS), LED45.4 (VSS), LED46.4 (VSS), LED47.4 (VSS), LED48.4 (VSS), LED49.4 (VSS), LED5.4 (VSS), LED50.4 (VSS), LED51.4 (VSS), LED52.4 (VSS), LED53.4 (VSS), LED54.4 (VSS), LED55.4 (VSS), LED56.4 (VSS), LED57.4 (VSS), LED58.4 (VSS), LED59.4 (VSS), LED6.4 (VSS), LED60.4 (VSS), LED61.4 (VSS), LED62.4 (VSS), LED63.4 (VSS), LED64.4 (VSS), LED65.4 (VSS), LED66.4 (VSS), LED67.4 (VSS), LED68.4 (VSS), LED69.4 (VSS), LED7.4 (VSS), LED8.4 (VSS), LED9.4 (VSS)
- net at LED36.2 (DOUT): now also LED37.4 (DIN); no longer LED37.3 (DIN)
- net at LED35.2 (DOUT): now also LED36.4 (DIN); no longer LED36.3 (DIN)
- net at LED6.2 (DOUT): now also LED7.4 (DIN); no longer LED7.3 (DIN)
- net at LED5.2 (DOUT): now also LED6.4 (DIN); no longer LED6.3 (DIN)
- net at LED21.2 (DOUT): now also LED22.4 (DIN); no longer LED22.3 (DIN)
- net at LED20.2 (DOUT): now also LED21.4 (DIN); no longer LED21.3 (DIN)
- net at LED65.2 (DOUT): now also LED66.4 (DIN); no longer LED66.3 (DIN)
- net at LED64.2 (DOUT): now also LED65.4 (DIN); no longer LED65.3 (DIN)
- net at LED54.2 (DOUT): now also LED55.4 (DIN); no longer LED55.3 (DIN)
- net at LED53.2 (DOUT): now also LED54.4 (DIN); no longer LED54.3 (DIN)
- net at LED60.2 (DOUT): now also LED61.4 (DIN); no longer LED61.3 (DIN)
- net at LED59.2 (DOUT): now also LED60.4 (DIN); no longer LED60.3 (DIN)
- net at LED29.2 (DOUT): now also LED30.4 (DIN); no longer LED30.3 (DIN)
- net at LED28.2 (DOUT): now also LED29.4 (DIN); no longer LED29.3 (DIN)
- net at LED46.2 (DOUT): now also LED47.4 (DIN); no longer LED47.3 (DIN)
- net at LED45.2 (DOUT): now also LED46.4 (DIN); no longer LED46.3 (DIN)
- net at LED37.2 (DOUT): now also LED38.4 (DIN); no longer LED38.3 (DIN)
- net at LED67.2 (DOUT): now also LED68.4 (DIN); no longer LED68.3 (DIN)
- net at LED66.2 (DOUT): now also LED67.4 (DIN); no longer LED67.3 (DIN)
- net at LED9.2 (DOUT): now also LED10.4 (DIN); no longer LED10.3 (DIN)
- net at LED8.2 (DOUT): now also LED9.4 (DIN); no longer LED9.3 (DIN)
- net at LED17.2 (DOUT): now also LED18.4 (DIN); no longer LED18.3 (DIN)
- net at LED16.2 (DOUT): now also LED17.4 (DIN); no longer LED17.3 (DIN)
- net at LED23.2 (DOUT): now also LED24.4 (DIN); no longer LED24.3 (DIN)
- net at LED22.2 (DOUT): now also LED23.4 (DIN); no longer LED23.3 (DIN)
- net at LED33.2 (DOUT): now also LED34.4 (DIN); no longer LED34.3 (DIN)
- net at LED32.2 (DOUT): now also LED33.4 (DIN); no longer LED33.3 (DIN)
- net at LED11.2 (DOUT): now also LED12.4 (DIN); no longer LED12.3 (DIN)
- net at LED10.2 (DOUT): now also LED11.4 (DIN); no longer LED11.3 (DIN)
- net at LED24.2 (DOUT): now also LED25.4 (DIN); no longer LED25.3 (DIN)
- net at LED25.2 (DOUT): now also LED26.4 (DIN); no longer LED26.3 (DIN)
- net at LED42.2 (DOUT): now also LED43.4 (DIN); no longer LED43.3 (DIN)
- net at LED41.2 (DOUT): now also LED42.4 (DIN); no longer LED42.3 (DIN)
- net at LED1.2 (DOUT): now also LED2.4 (DIN); no longer LED2.3 (DIN)
- net at LED14.2 (DOUT): now also LED15.4 (DIN); no longer LED15.3 (DIN)
- net at LED13.2 (DOUT): now also LED14.4 (DIN); no longer LED14.3 (DIN)
- net at LED31.2 (DOUT): now also LED32.4 (DIN); no longer LED32.3 (DIN)
- net at LED68.2 (DOUT): now also LED69.4 (DIN); no longer LED69.3 (DIN)
- net at LED58.2 (DOUT): now also LED59.4 (DIN); no longer LED59.3 (DIN)
- net at LED40.2 (DOUT): now also LED41.4 (DIN); no longer LED41.3 (DIN)
- net at LED39.2 (DOUT): now also LED40.4 (DIN); no longer LED40.3 (DIN)
- net at LED18.2 (DOUT): now also LED19.4 (DIN); no longer LED19.3 (DIN)
- net at LED63.2 (DOUT): now also LED64.4 (DIN); no longer LED64.3 (DIN)
- net at LED57.2 (DOUT): now also LED58.4 (DIN); no longer LED58.3 (DIN)
- net at LED3.2 (DOUT): now also LED4.4 (DIN); no longer LED4.3 (DIN)
- net at LED2.2 (DOUT): now also LED3.4 (DIN); no longer LED3.3 (DIN)
- net at LED43.2 (DOUT): now also LED44.4 (DIN); no longer LED44.3 (DIN)
- net at LED19.2 (DOUT): now also LED20.4 (DIN); no longer LED20.3 (DIN)
- net at LED44.2 (DOUT): now also LED45.4 (DIN); no longer LED45.3 (DIN)
- net at LED4.2 (DOUT): now also LED5.4 (DIN); no longer LED5.3 (DIN)
- net at LED51.2 (DOUT): now also LED52.4 (DIN); no longer LED52.3 (DIN)
- net at LED50.2 (DOUT): now also LED51.4 (DIN); no longer LED51.3 (DIN)
- net at LED34.2 (DOUT): now also LED35.4 (DIN); no longer LED35.3 (DIN)
- net at LED62.2 (DOUT): now also LED63.4 (DIN); no longer LED63.3 (DIN)
- net at LED61.2 (DOUT): now also LED62.4 (DIN); no longer LED62.3 (DIN)
- net at LED12.2 (DOUT): now also LED13.4 (DIN); no longer LED13.3 (DIN)
- net at LED7.2 (DOUT): now also LED8.4 (DIN); no longer LED8.3 (DIN)
- net at LED56.2 (DOUT): now also LED57.4 (DIN); no longer LED57.3 (DIN)
- net at LED55.2 (DOUT): now also LED56.4 (DIN); no longer LED56.3 (DIN)
- net at LED48.2 (DOUT): now also LED49.4 (DIN); no longer LED49.3 (DIN)
- net at LED47.2 (DOUT): now also LED48.4 (DIN); no longer LED48.3 (DIN)
- net at LED15.2 (DOUT): now also LED16.4 (DIN); no longer LED16.3 (DIN)
- net at LED30.2 (DOUT): now also LED31.4 (DIN); no longer LED31.3 (DIN)
- net at LED49.2 (DOUT): now also LED50.4 (DIN); no longer LED50.3 (DIN)
- net at LED26.2 (DOUT): now also LED27.4 (DIN); no longer LED27.3 (DIN)
- net at LED52.2 (DOUT): now also LED53.4 (DIN); no longer LED53.3 (DIN)
- net at LED38.2 (DOUT): now also LED39.4 (DIN); no longer LED39.3 (DIN)
- net at LED27.2 (DOUT): now also LED28.4 (DIN); no longer LED28.3 (DIN)
